Commit message: continuous joints+ param

File: src/my_robot_description/urdf/rubot/rubot_mecanum_custom.urdf (robot description, URDF)
Before this commit: robot rubot, 9 links, 8 joints
Joints:
- joint base_link_joint: type fixed -> continuous
- joint joint_camera: type fixed -> continuous
- joint joint_part: type fixed -> continuous
- joint scan_joint: type fixed -> continuous

Commit message: fix joints

File: src/my_robot_description/urdf/rubot/rubot_mecanum_custom.urdf (robot description, URDF)
Before this commit: robot rubot_mecanum_custom, 9 links, 8 joints
Joints:
- joint joint_camera: type continuous -> fixed
- joint joint_part: type continuous -> fixed
- joint scan_joint: type continuous -> fixed

Commit message: correction custom urdf

File: src/my_robot_description/urdf/rubot/rubot_mecanum_custom.urdf (robot description, URDF)
Before this commit: robot rubot_mecanum_custom, 9 links, 8 joints
Joints:
- joint base_link_joint: type continuous -> fixed
- joint joint_camera: type continuous -> fixed
- joint joint_part: type continuous -> fixed
- joint scan_joint: type continuous -> fixed
